File: Hardware/rising_sun_power_board/rising_sun_power_board.kicad_pcb (KiCad board)
At the start: 2 copper layers, 30 parts, among them J1 POWER_IN, J2 Conn_01x03_Socket, J3 Conn_01x03_Socket, SW1 SW_Push, SW2 SW_Push, U1 ESP32, U2 MIC5219, U3 UA78M05IDCYR, U4 TXU0102DCUR

Commit message: layout le done
Parts:
- removed U3: UA78M05IDCYR, Package_TO_SOT_SMD:SOT-223-3_TabPin2
- added C7: 1uF, Capacitor_SMD:C_0603_1608Metric, B.Cu at (64.9, 55.9)
- added G***: LOGO, custom_footprints:teehee, B.Cu at (80.0, 46.4)
- added U5: UA78M05IDCYR, Package_TO_SOT_SMD:SOT-223, B.Cu at (60.5, 47.2)
- C1, C2, C3, C4, C5, C6, D1, D2, D3, D4, D5, R1, R2, R3, R4, R5, R6, R7, SW1, SW2, U2, U4: moved to B.Cu
- J1: value POWER_IN -> Barrel_Jack_MountingPin; footprint Connector_BarrelJack:BarrelJack_Wuerth_6941xx301002 -> custom_footprints:CUI_PJ-202A
- moved R4 70.0 mm to (55.1, 26.7), turned to 180 degrees
- moved R7 69.6 mm to (55.1, 24.1), turned to 180 degrees
- moved U4 63.6 mm to (68.6, 33.7), turned to -90 degrees
- moved C5 60.6 mm to (68.6, 30.5), turned to 180 degrees
- moved R5 59.9 mm to (55.1, 30.5), turned to 180 degrees
- moved R6 58.9 mm to (55.1, 34.3), turned to 180 degrees
- moved SW2 57.9 mm to (85.1, 17.8), turned to 90 degrees
- moved D4 54.1 mm to (58.4, 30.5)
- moved D5 53.1 mm to (58.4, 34.3)
- moved J2 52.0 mm to (79.2, 40.5)
- moved C6 49.3 mm to (66.0, 34.3), turned to 90 degrees
- moved U2 47.8 mm to (62.7, 58.7), turned to 180 degrees
- moved C3 45.1 mm to (65.4, 42.5)
- moved J3 45.0 mm to (79.2, 55.1)
- moved SW1 43.2 mm to (85.1, 26.0), turned to 90 degrees
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Connections:
- R7 pad 2: /GPIO_BUTTON12 -> /GPIO_BUTTON2
- SW2 pad 1: /GPIO_BUTTON12 -> /GPIO_BUTTON2
Routing:
- net /GPIO_BUTTON2: track 0.00 -> 44.1 mm, vias 0 -> 2
- net /GPIO_BUTTON1: track 0.00 -> 42.5 mm, vias 0 -> 2
- net GND: track 0.00 -> 41.5 mm, vias 0 -> 19
- net /LED_ENABLE_5V_2: track 0.00 -> 40.7 mm, vias 0 -> 3
- net /5V_Enable: track 0.00 -> 31.9 mm, vias 0 -> 2
- net /LEVEL_SHIFT_EN: track 0.00 -> 17.5 mm, vias 0 -> 2
- net +3V3: track 0.00 -> 15.4 mm, vias 0 -> 8
- net /LED_ENABLE_5V_1: track 0.00 -> 14.9 mm, vias 0 -> 1
- net /LED_ENABLE_3V3_2: track 0.00 -> 14.8 mm
- net /LED_ENABLE_3V3_1: track 0.00 -> 11.3 mm
- net +5V: track 0.00 -> 8.72 mm, vias 0 -> 5
- net /GPIO_LED2: track 0.00 -> 4.38 mm
- net /GPIO_LED1: track 0.00 -> 3.85 mm
- net Net-(D3-K): track 0.00 -> 2.64 mm
- net Net-(D2-K): track 0.00 -> 2.64 mm
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- added copper zone on B.Cu, net +12V
- added copper zone on In2.Cu, net +3V3
- added copper zone on F.Cu, net +5V
- added copper zone on B.Cu, net GND
- added copper zone on In1.Cu, net GND
Other:
- board outline added: 38.1 x 63.5 mm
- copper layers 2 -> 4

Commit message: :octocat: Fixed layout and gpio assignment
Parts:
- moved J3 15.9 mm to (79.2, 39.2)
- moved J2 12.1 mm to (79.2, 52.5)
- moved TP1 1.91 mm to (65.4, 75.6)
- moved TP2 1.91 mm to (60.3, 75.6)
- moved TP3 1.91 mm to (55.2, 75.6)
- moved SW1 0.42 mm to (84.7, 26.0)
- moved SW2 0.42 mm to (84.7, 17.8)
Connections:
- U1 pad 28: unconnected-(U1-4-Pad28) -> /5V_Enable
- U1 pad 30: /LEVEL_SHIFT_EN -> unconnected-(U1-2-Pad30)
- U1 pad 31: /LED_ENABLE_3V3_2 -> unconnected-(U1-15-Pad31)
- U1 pad 32: /LED_ENABLE_3V3_1 -> unconnected-(U1-5-Pad32)
- U1 pad 33: /5V_Enable -> unconnected-(U1-18-Pad33)
- U1 pad 34: unconnected-(U1-23-Pad34) -> /LED_ENABLE_3V3_2
- U1 pad 35: unconnected-(U1-19-Pad35) -> /LEVEL_SHIFT_EN
- U1 pad 36: unconnected-(U1-22-Pad36) -> /LED_ENABLE_3V3_1
Routing:
- net /5V_Enable: track 31.9 -> 14.0 mm
- net /LED_ENABLE_5V_1: track 14.9 -> 30.3 mm, vias 1 -> 3
- net /LED_ENABLE_5V_2: track 40.7 -> 26.2 mm
- net /LEVEL_SHIFT_EN: track 17.5 -> 5.96 mm, vias 2 -> 0
- net GND: track 41.5 -> 33.9 mm
- net /LED_ENABLE_3V3_1: track 11.3 -> 4.60 mm
- net /LED_ENABLE_3V3_2: track 14.8 -> 8.94 mm
- net /GPIO_BUTTON1: track 42.5 -> 44.4 mm
- net +5V: track 8.72 -> 9.56 mm
Other:
- board text added: "Lina Lin Wei & Ian Ballou"
