File: Hardware/rising_sun_power_board/rising_sun_power_board.kicad_sch (KiCad schematic)
At the start: 30 parts, among them J1 POWER_IN, J2 Conn_01x03_Socket, J3 Conn_01x03_Socket, SW201 SW_Push, U1 ESP32, U2 MIC5219, U3 UA78M05IDCYR, U4 TXU0102DCUR

Commit message: layout le done
Parts:
- removed J1: POWER_IN, Connector_BarrelJack:BarrelJack_Wuerth_6941xx301002, symbol Connector:Barrel_Jack
- removed U3: UA78M05IDCYR, Package_TO_SOT_SMD:SOT-223-3_TabPin2, symbol Regulator_Linear:AMS1117-3.3
- added C7: 1uF, Capacitor_SMD:C_0603_1608Metric, symbol Device:C_Small
- added J1: Barrel_Jack_MountingPin, custom_footprints:CUI_PJ-202A, symbol Connector:Barrel_Jack_MountingPin
- added U5: UA78M05IDCYR, Package_TO_SOT_SMD:SOT-223, symbol customLibrary:uA78M33
Connections:
- net GPIO_BUTTON12 is gone; now on net GPIO_BUTTON2: R212.2, SW201.1
- net +12V: now also C7.2, J1.1, U5.1 (INPUT)
- net +3V3: now also U5.3 (OUTPUT)
- net GND: now also C7.1, J1.2, U5.2 (GND), U5.4 (GND)
- no-connect marks 25 -> 26
Other:
- moved on the sheet: C1, C2, C3, C4, D205, D206, R212, R213, R214, SW201, U1, U2

Commit message: :octocat: Fixed layout and gpio assignment
Connections:
- net 5V_Enable: now also U1.28 (4); no longer U1.33 (18)
- net LED_ENABLE_3V3_1: now also U1.36 (22); no longer U1.32 (5)
- net LED_ENABLE_3V3_2: now also U1.34 (23); no longer U1.31 (15)
- net LEVEL_SHIFT_EN: now also U1.35 (19); no longer U1.30 (2)
Other:
- note added: "Input only GPIO:34, 35, 36, 37, 38, 39 For flash/PSRAM:16, 17 Has other important functions:0, 2, 5"
Changed lines of the file:
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@@
   )
   (no_connect (at 113.03 67.945))
-  (no_connect (at 146.05 45.085))
+  (no_connect (at 146.05 52.705))
   (no_connect (at 146.05 78.105))
-  (no_connect (at 146.05 42.545))
+  (no_connect (at 146.05 50.165))
   (no_connect (at 146.05 37.465))
   (no_connect (at 146.05 65.405))
@@
   (no_connect (at 146.05 60.325))
   (no_connect (at 146.05 67.945))
-  (no_connect (at 146.05 47.625))
+  (no_connect (at 146.05 55.245))
   (no_connect (at 146.05 34.925))
   (no_connect (at 113.03 55.245))
+  (no_connect (at 146.05 57.785))
   (no_connect (at 113.03 57.785))
   (no_connect (at 113.03 62.865))
   (no_connect (at 113.03 42.545))
-  (no_connect (at 146.05 62.865))
   (no_connect (at 49.53 40.005))
   (no_connect (at 146.05 40.005))
@@
     (stroke (width 0) (type default))
   )
-  (wire (pts (xy 146.05 55.245) (xy 149.86 55.245))
+  (wire (pts (xy 146.05 45.085) (xy 149.86 45.085))
     (stroke (width 0) (type default))
   )
@@
     (stroke (width 0) (type default))
   )
-  (wire (pts (xy 146.05 57.785) (xy 149.86 57.785))
+  (wire (pts (xy 146.05 47.625) (xy 149.86 47.625))
     (stroke (width 0) (type default))
   )
@@
     (stroke (width 0) (type default))
   )
-  (wire (pts (xy 146.05 52.705) (xy 149.86 52.705))
+  (wire (pts (xy 146.05 42.545) (xy 149.86 42.545))
     (stroke (width 0) (type default))
   )
@@
     (stroke (width 0) (type default))
   )
-  (wire (pts (xy 149.86 50.165) (xy 146.05 50.165))
+  (wire (pts (xy 149.86 62.865) (xy 146.05 62.865))
     (stroke (width 0) (type default))
   )
@@
     (stroke (width 0) (type default))
   )
+  (text "Input only GPIO:34, 35, 36, 37, 38, 39\nFor flash/PSRAM:16, 17\nHas other important functions:0, 2, 5"
+    (at 161.29 31.115 0)
+    (effects (font (size 1.27 1.27)) (justify left bottom))
+  )
   (text "02/02/2024" (at 206.375 194.31 0)
     (effects (font (size 1.27 1.27)) (justify left bottom))
@@
     (effects (font (size 1.27 1.27)) (justify right bottom))
   )
-  (label "5V_Enable" (at 149.86 50.165 0) (fields_autoplaced)
+  (label "5V_Enable" (at 149.86 62.865 0) (fields_autoplaced)
     (effects (font (size 1.27 1.27)) (justify left bottom))
   )
@@
     (effects (font (size 1.27 1.27)) (justify right bottom))
   )
-  (label "LEVEL_SHIFT_EN" (at 149.86 57.785 0) (fields_autoplaced)
+  (label "LEVEL_SHIFT_EN" (at 149.86 45.085 0) (fields_autoplaced)
     (effects (font (size 1.27 1.27)) (justify left bottom))
   )
@@
     (effects (font (size 1.27 1.27)) (justify left bottom))
   )
-  (label "LED_ENABLE_3V3_2" (at 149.86 55.245 0) (fields_autoplaced)
+  (label "LED_ENABLE_3V3_2" (at 149.86 47.625 0) (fields_autoplaced)
     (effects (font (size 1.27 1.27)) (justify left bottom))
   )
@@
     (effects (font (size 1.27 1.27)) (justify right bottom))
   )
-  (label "LED_ENABLE_3V3_1" (at 149.86 52.705 0) (fields_autoplaced)
-    (effects (font (size 1.27 1.27)) (justify left bottom))
-  )
+  (label "LED_ENABLE_3V3_1" (at 149.86 42.545 0) (fields_autoplaced)
+    (effects (font (size 1.27 1.27)) (justify left bottom))
+  )
